File: pcbservo-dc/pcbservo-dc.kicad_sch (KiCad schematic)
At the start: 29 parts, among them J10 Conn_01x03, J12 Conn_01x02, J13 Conn_01x02, J4 Conn_01x03, J5 Conn_01x03, SW1 SW_Nidec_CAS-120A1, SW2 SW_Nidec_CAS-120A1, SW3 SW_Nidec_CAS-120A1, SW4 SW_Nidec_CAS-120A1, SW5 SW_Nidec_CAS-120A1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

Commit message: résolution des erreurs
Other:
- moved on the sheet: C3, C4, C5, C6, Driver1, J12, J13, SW1, SW2, SW3, SW4, SW5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
