File: pcbservo-dc/untitled.kicad_sch (KiCad schematic)
At the start: 36 parts, among them IC1 NC7WZ241K8X, IC2 NC7WZ241K8X, IC3 NC7WZ241K8X, J7 Conn_ST_STDC14, J8 Conn_01x03, U7 STM32H573RITx

Commit message: résolution des erreurs
Other:
- moved on the sheet: C10, C11, C12, C13, C14, C25, C26, C27, C7, C8, C9, L1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
