File: pcbservo-dc/untitled.kicad_sch1.kicad_sch (KiCad schematic)
At the start: 21 parts, among them J1 Conn_01x02, J14 R-78B5.0-2.0, J2 Conn_01x02, J3 BU33SD5WG-TR

Commit message: résolution des erreurs
Parts:
- TP1, TP2: footprint TestPoint:TestPoint_Pad_D2.0mm -> TestPoint:TestPoint_Pad_D1.0mm
Connections:
- net +25V: now also J14.1 (IN)
- net +6V: no longer J14.1 (IN)
Other:
- note added: "regulateur 5V à 3,3 V"
- note added: "regulateur de 25V à 5V"
- note removed: "regulateur 6V à 3,3 V"
- note removed: "regulateur de 6V à 5V"
Changed lines of the file:
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@@
 	(rectangle
 		(start 14.605 84.455)
-		(end 86.36 128.27)
+		(end 101.092 135.636)
 		(stroke
 			(width 0)
@@
 		)
 	)
-	(text "regulateur 6V à 3,3 V\n"
+	(text "regulateur 5V à 3,3 V\n"
 		(exclude_from_sim no)
 		(at 27.178 17.018 0)
@@
 		)
 	)
-	(text "regulateur de 6V à 5V\n"
+	(text "regulateur de 25V à 5V\n"
 		(exclude_from_sim no)
 		(at 27.686 86.868 0)
@@
 	(wire
 		(pts
-			(xy 39.37 109.22) (xy 43.18 109.22)
+			(xy 31.75 109.22) (xy 43.18 109.22)
 		)
 		(stroke
@@
 			)
 		)
-		(property "Footprint" "TestPoint:TestPoint_Pad_D2.0mm"
+		(property "Footprint" "TestPoint:TestPoint_Pad_D1.0mm"
 			(at 69.85 109.22 0)
 			(effects
@@
 	)
 	(symbol
+		(lib_id "power:+7.5V")
+		(at 31.75 109.22 0)
+		(unit 1)
+		(exclude_from_sim no)
+		(in_bom yes)
+		(on_board yes)
+		(dnp no)
+		(fields_autoplaced yes)
+		(property "Reference" "#PWR054"
+			(at 31.75 113.03 0)
+			(effects
+				(font
+					(size 1.27 1.27)
+				)
+				(hide yes)
+			)
+		)
+		(property "Value" "+25V"
+			(at 34.29 107.9499 0)
+			(effects
+				(font
+					(size 1.27 1.27)
+				)
+				(justify left)
+			)
+		)
+		(property "Footprint" ""
+			(at 31.75 109.22 0)
+			(effects
+				(font
+					(size 1.27 1.27)
+				)
+				(hide yes)
+			)
+		)
+		(property "Datasheet" ""
+			(at 31.75 109.22 0)
+			(effects
+				(font
+					(size 1.27 1.27)
+				)
+				(hide yes)
+			)
+		)
+		(property "Description" "Power symbol creates a global label with name \"+7.5V\""
+			(at 31.75 109.22 0)
+			(effects
+				(font
+					(size 1.27 1.27)
+				)
+				(hide yes)
+			)
+		)
+		(pin "1"
+		)
+		(instances
+			(project "pcbservo-dc"
+				(path "/be41f19f-3f75-42cb-bbbf-7251912cb437/634157a2-b1a1-4f11-8683-17550dacecc7"
+					(reference "#PWR054")
+					(unit 1)
+				)
+			)
+		)
+	)
+	(symbol
 		(lib_name "GND_3")
 		(lib_id "power:GND")
@@
 			)
 		)
-		(property "Footprint" "TestPoint:TestPoint_Pad_D2.0mm"
+		(property "Footprint" "TestPoint:TestPoint_Pad_D1.0mm"
 			(at 76.2 50.8 0)
 			(effects
@@
 					(unit 1)
 				)
-			)
-		)
-	)
-	(symbol
-		(lib_id "power:+7.5V")
-		(at 39.37 109.22 0)
-		(unit 1)
-		(exclude_from_sim no)
-		(in_bom yes)
-		(on_board yes)
-		(dnp no)
-		(fields_autoplaced yes)
-		(property "Reference" "#PWR041"
-			(at 39.37 113.03 0)
-			(effects
-				(font
-					(size 1.27 1.27)
-				)
-				(hide yes)
-			)
-		)
-		(property "Value" "+6V"
-			(at 39.37 104.14 0)
-			(effects
-				(font
-					(size 1.27 1.27)
-				)
-			)
-		)
-		(property "Footprint" ""
-			(at 39.37 109.22 0)
-			(effects
-				(font
-					(size 1.27 1.27)
-				)
-				(hide yes)
-			)
-		)
-		(property "Datasheet" ""
-			(at 39.37 109.22 0)
-			(effects
-				(font
-					(size 1.27 1.27)
-				)
-				(hide yes)
-			)
-		)
-		(property "Description" "Power symbol creates a global label with name \"+7.5V\""
-			(at 39.37 109.22 0)
-			(effects
-				(font
-					(size 1.27 1.27)
-				)
-				(hide yes)
-			)
-		)
-		(pin "1"
-		)
-		(instances
-			(project "pcbservo-dc"
-				(path "/be41f19f-3f75-42cb-bbbf-7251912cb437/634157a2-b1a1-4f11-8683-17550dacecc7"
-					(reference "#PWR041")
-					(unit 1)
-				)
